Commit message: Add lidar & ros controller in gazebo

File: src/simulation/description/robot.urdf.xacro (robot description, xacro)
@@ -2,3 +2,6 @@
 <robot name="Ollie" xmlns:xacro="http://www.ros.org/wiki/xacro">
     <xacro:include filename="robot_core.xacro"/>
+    <!-- <xacro:include filename="gazebo_control.xacro"/> -->
+    <xacro:include filename="lidar.xacro"/>
+    <xacro:include filename="ros2_control.xacro"/>
 </robot>

File: src/simulation/description/robot_core.xacro (robot description, xacro)
@@ -13,5 +13,5 @@
     <xacro:property name="caster_radius" value="0.01"/>
     <xacro:property name="caster_wheel_mass" value="0.02"/>
-    <xacro:property name="caster_wheel_offset_x" value="0.15"/>
+    <xacro:property name="caster_wheel_offset_x" value="0.11"/>
     <material name="white">
         <color rgba="1 1 1 1" />
@@ -55,4 +55,7 @@
         </xacro:inertial_box>
     </link>
+    <gazebo reference="chassis_link">
+        <material>Gazebo/White</material>
+    </gazebo>
     <!-- WHEELS -->
     <joint name="left_wheel_joint" type="continuous">
@@ -78,4 +81,7 @@
         </xacro:inertial_cylinder>
     </link>
+    <gazebo reference="left_wheel_link">
+        <material>Gazebo/Black</material>
+    </gazebo>
     <joint name="right_wheel_joint" type="continuous">
         <parent link="base_link"/>
@@ -100,4 +106,7 @@
         </xacro:inertial_cylinder>
     </link>
+    <gazebo reference="right_wheel_link">
+        <material>Gazebo/Black</material>
+    </gazebo>
     <!-- CASTER WHEEL -->
     <joint name="caster_wheel_joint" type="fixed">
@@ -122,3 +131,8 @@
         </xacro:inertial_sphere>
     </link>
+    <gazebo reference="caster_wheel_link">
+        <material>Gazebo/Black</material>
+        <mu1>0.0001</mu1>
+        <mu2>0.0002</mu2>
+    </gazebo>
 </robot>
