Commit message: Add SLAM mapping

File: src/simulation/description/lidar.xacro (robot description, xacro)
@@ -3,8 +3,8 @@
     <joint name="laser_joint" type="fixed">
         <parent link="chassis_link"/>
-        <child link="laser_link"/>
+        <child link="laser_frame"/>
         <origin xyz="0.1 0.0 0.02" rpy="0.0 0.0 0.0"/>
     </joint>
-    <link name="laser_link">
+    <link name="laser_frame">
         <visual>
             <geometry>
@@ -22,5 +22,5 @@
         </xacro:inertial_cylinder>
     </link>
-    <gazebo reference="laser_link">
+    <gazebo reference="laser_frame">
         <material>Gazebo/Red</material>
         <sensor name="laser" type="ray">

File: src/simulation/description/robot_core.xacro (robot description, xacro)
@@ -31,4 +31,10 @@
     <!--  BASE LINK -->
     <link name="base_link"></link>
+    <joint name="base_footprint_joint" type="fixed">
+        <parent link="base_link"/>
+        <child link="base_footprint"/>
+        <origin xyz="0 0 0" rpy="0 0 0"/>
+    </joint>
+    <link name="base_footprint"></link>
     <!-- CHASSIS LINK -->
     <joint name="chassis_joint" type="fixed">
@@ -74,5 +80,6 @@
         <collision>
             <geometry>
-                <cylinder radius="${wheel_radius}" length="${wheel_thickness}"/>
+                <!-- Changed length to prevent wheel slippage -->
+                <cylinder radius="${wheel_radius}" length="0.0001"/>
             </geometry>
         </collision>
@@ -99,5 +106,6 @@
         <collision>
             <geometry>
-                <cylinder radius="${wheel_radius}" length="${wheel_thickness}"/>
+                <!-- Changed length to prevent wheel slippage -->
+                <cylinder radius="${wheel_radius}" length="0.0001"/>
             </geometry>
         </collision>
